Commit message: Different Types of Joints in URDF

File: my_robot.urdf (robot description, URDF)
Before this commit: robot my_robot, 3 links, 2 joints
Links:
- removed link third_link
Joints:
- removed joint second_third_joint
- joint base_second_joint: axis (none) -> 1 0 0; limit (none) -> lower=0.0 upper=0.2 effort=100 velocity=100; type fixed -> prismatic

Commit message: Add a Wheel to the Robot

File: my_robot.urdf (robot description, URDF)
Before this commit: robot my_robot, 2 links, 1 joints
Links:
- removed link second_link
- added link right_wheel_link; visual cylinder length=0.05 radius=0.1
Joints:
- removed joint base_second_joint
- added joint base_right_wheel_joint: type continuous, parent base_link, child right_wheel_link, origin xyz=-0.15 -0.225 0 rpy=0 0 0, axis 0 1 0

Commit message: Activity 1

File: my_robot.urdf (robot description, URDF)
Before this commit: robot my_robot, 2 links, 1 joints
Links:
- added link base_footprint
- added link caster_wheel_link; visual sphere radius=0.05
- added link left_wheel_link; visual cylinder length=0.05 radius=0.1
Joints:
- added joint base_caster_wheel_joint: type fixed, parent base_link, child caster_wheel_link, origin xyz=0.2 0 -0.05 rpy=0 0 0
- added joint base_joint: type fixed, parent base_footprint, child base_link, origin xyz=0 0 0.1 rpy=0 0 0
- added joint base_left_wheel_joint: type continuous, parent base_link, child left_wheel_link, origin xyz=-0.15 -0.225 0 rpy=0 0 0, axis 0 1 0
- joint base_right_wheel_joint: origin xyz=-0.15 -0.225 0 rpy=0 0 0 -> xyz=-0.15 0.225 0 rpy=0 0 0
